Commit message: 9/11

File: description/gz_diff_drive_control.xacro (robot description, xacro)
@@ -7,5 +7,5 @@
             <left_joint>left_wheel_joint</left_joint>
             <right_joint>right_wheel_joint</right_joint>
-            <wheel_separation>0.222</wheel_separation>
+            <wheel_separation>0.2283</wheel_separation>
             <wheel_radius>0.034</wheel_radius>
             <!-- Limits -->

File: description/robot_main.xacro (robot description, xacro)
@@ -3,5 +3,5 @@
     <xacro:include filename = "inertial_macros.xacro" />
     <xacro:property name="chassis_length"           value="0.263"/>
-    <xacro:property name="chassis_width"            value="0.18"/>
+    <xacro:property name="chassis_width"            value="0.19"/>
     <xacro:property name="chassis_height"           value="0.1"/>
     <xacro:property name="chassis_mass"             value="0.700"/>
@@ -10,5 +10,6 @@
     <xacro:property name="wheel_mass"               value="0.050"/>
     <xacro:property name="wheel_offset_x"           value="0.075"/>
-    <xacro:property name="wheel_offset_y"           value="0.11"/>
+    <!-- <xacro:property name="wheel_offset_y"           value="0.105"/> -->
+    <xacro:property name="wheel_offset_y"           value="0.114"/>
     <xacro:property name="wheel_offset_z"           value="0.015"/>
     <xacro:property name="caster_wheel_radius"      value="${wheel_radius - wheel_offset_z}"/>
@@ -55,5 +56,5 @@
             </geometry>
         </collision>
-        <xacro:inertial_box mass= "0.5" x="${chassis_length}" y="${chassis_width}" z="${chassis_height}">
+        <xacro:inertial_box mass= "0.7" x="${chassis_length}" y="${chassis_width}" z="${chassis_height}">
             <origin xyz= "${chassis_length/2} 0 ${chassis_height/2}" rpy= "0 0 0"/>
         </xacro:inertial_box>

File: description/ros2_control.xacro (robot description, xacro)
@@ -8,10 +8,9 @@
                     <param name="left_wheel_name">left_wheel_joint</param>
                     <param name="right_wheel_name">right_wheel_joint</param>
-                    <param name="loop_rate">30</param>
+                    <param name="loop_rate">50</param>
                     <param name="device">/dev/ttyUSB0</param>
                     <param name="baud_rate">57600</param>
                     <param name="timeout">1000</param>
-                    <!-- <param name="enc_counts_per_rev">3450</param>  -->
-                    <param name="enc_counts_per_rev">1975</param>
+                    <param name="enc_counts_per_rev">1976</param>
             </hardware>
             <joint name="left_wheel_joint">
