Commit message: save local changes before pull

File: description/robot_main.xacro (robot description, xacro)
@@ -10,6 +10,5 @@
     <xacro:property name="wheel_mass"               value="0.050"/>
     <xacro:property name="wheel_offset_x"           value="0.075"/>
-    <!-- <xacro:property name="wheel_offset_y"           value="0.105"/> -->
-    <xacro:property name="wheel_offset_y"           value="0.114"/>
+    <xacro:property name="wheel_offset_y"           value="0.105"/>
     <xacro:property name="wheel_offset_z"           value="0.015"/>
     <xacro:property name="caster_wheel_radius"      value="${wheel_radius - wheel_offset_z}"/>
@@ -56,5 +55,5 @@
             </geometry>
         </collision>
-        <xacro:inertial_box mass= "0.7" x="${chassis_length}" y="${chassis_width}" z="${chassis_height}">
+        <xacro:inertial_box mass= "0.5" x="${chassis_length}" y="${chassis_width}" z="${chassis_height}">
             <origin xyz= "${chassis_length/2} 0 ${chassis_height/2}" rpy= "0 0 0"/>
         </xacro:inertial_box>

File: description/ros2_control.xacro (robot description, xacro)
@@ -12,4 +12,5 @@
                     <param name="baud_rate">57600</param>
                     <param name="timeout">1000</param>
+                    <!-- <param name="enc_counts_per_rev">3450</param>  -->
                     <param name="enc_counts_per_rev">1976</param>
             </hardware>

Commit message: Cập nhật

File: description/robot_main.xacro (robot description, xacro)
@@ -10,5 +10,5 @@
     <xacro:property name="wheel_mass"               value="0.050"/>
     <xacro:property name="wheel_offset_x"           value="0.075"/>
-    <xacro:property name="wheel_offset_y"           value="0.105"/>
+    <xacro:property name="wheel_offset_y"           value="0.114"/>
     <xacro:property name="wheel_offset_z"           value="0.015"/>
     <xacro:property name="caster_wheel_radius"      value="${wheel_radius - wheel_offset_z}"/>
