Commit message: sửa file xacro

File: description/lidar.xacro (robot description, xacro)
@@ -3,11 +3,11 @@
     <xacro:property name="lidar_radius"             value="0.025"/>
     <xacro:property name="lidar_thickness"          value="0.040"/>
-    <xacro:property name="lidar_offset_x"           value="0.230"/>
-    <xacro:property name="lidar_offset_z"           value="0.098"/>
+    <xacro:property name="lidar_offset_x"           value="0.208"/>
+    <xacro:property name="lidar_offset_z"           value="0.12"/>
     <!-- Lidar -->
     <joint name="lidar_joint" type="fixed">
         <parent link="chasis"/>
         <child link="lidar_frame"/>
-        <origin xyz="${lidar_offset_x} 0.0 ${lidar_offset_z}" rpy="0 0 ${pi}"/>
+        <origin xyz="${lidar_offset_x} 0.0 ${lidar_offset_z}" rpy="0 0 0"/>
     </joint>
     <link name="lidar_frame">
@@ -16,5 +16,5 @@
                 <cylinder radius="${lidar_radius}" length="${lidar_thickness}"/>
             </geometry>
-            <material name="orange"/>
+            <material name="black"/>
         </visual>
         <collision>

File: description/robot_main.xacro (robot description, xacro)
@@ -2,6 +2,6 @@
 <robot xmlns:xacro="http://www.ros.org/wiki/xacro">
     <xacro:include filename = "inertial_macros.xacro" />
-    <xacro:property name="chassis_length"           value="0.27"/>
-    <xacro:property name="chassis_width"            value="0.185"/>
+    <xacro:property name="chassis_length"           value="0.263"/>
+    <xacro:property name="chassis_width"            value="0.18"/>
     <xacro:property name="chassis_height"           value="0.1"/>
     <xacro:property name="chassis_mass"             value="0.700"/>
@@ -9,7 +9,7 @@
     <xacro:property name="wheel_thickness"          value="0.026"/>
     <xacro:property name="wheel_mass"               value="0.050"/>
-    <xacro:property name="wheel_offset_x"           value="0.133"/>
-    <xacro:property name="wheel_offset_y"           value="0.133"/>
-    <xacro:property name="wheel_offset_z"           value="0.020"/>
+    <xacro:property name="wheel_offset_x"           value="0.075"/>
+    <xacro:property name="wheel_offset_y"           value="0.11"/>
+    <xacro:property name="wheel_offset_z"           value="0.015"/>
     <xacro:property name="caster_wheel_radius"      value="${wheel_radius - wheel_offset_z}"/>
     <xacro:property name="caster_wheel_mass"        value="0.010"/>
@@ -22,13 +22,4 @@
     <material name="black">
         <color rgba= "0 0 0 1"/>
-    </material>
-    <material name= "orange">
-        <color rgba= "1 0.25 0 1"/>
-    </material>
-    <material name="cyan">
-        <color rgba= "0 1 1 1"/>
-    </material>
-    <material name="indigo">
-        <color rgba= "0.294 0 0.51 1"/>
     </material>
     <!-- convention (except base_link): joint followed by link -->
@@ -56,5 +47,5 @@
                 <box size = "${chassis_length} ${chassis_width} ${chassis_height}"/>
             </geometry>
-            <material name= "black"/>
+            <material name= "white"/>
         </visual>
         <collision>
@@ -69,5 +60,5 @@
     </link>
     <gazebo reference="chasis">
-        <material>Gazebo/Black</material>
+        <material>Gazebo/White</material>
     </gazebo>
     <!-- left_wheel -->
@@ -83,5 +74,5 @@
                 <cylinder radius = "${wheel_radius}" length= "${wheel_thickness}"/>
             </geometry>
-            <material name= "orange"/>
+            <material name= "black"/>
         </visual>
         <collision>
@@ -95,5 +86,5 @@
     </link>
     <gazebo reference="left_wheel">
-        <material>Gazebo/Orange</material>
+        <material>Gazebo/Black</material>
     </gazebo>
     <!-- right_wheel -->
@@ -109,5 +100,5 @@
                 <cylinder radius = "${wheel_radius}" length= "${wheel_thickness}"/>
             </geometry>
-            <material name= "orange"/>
+            <material name= "black"/>
         </visual>
         <collision>
@@ -121,5 +112,5 @@
     </link>
     <gazebo reference="right_wheel">
-        <material>Gazebo/Orange</material>
+        <material>Gazebo/Black</material>
     </gazebo>
     <!-- caster_wheel -->
@@ -134,5 +125,5 @@
                 <sphere radius = "${caster_wheel_radius}"/>
             </geometry>
-            <material name= "orange"/>
+            <material name= "white"/>
         </visual>
         <collision>
@@ -146,5 +137,5 @@
     </link>
     <gazebo reference="caster_wheel">
-        <material>Gazebo/Orange</material>
+        <material>Gazebo/White</material>
         <mu1 value= "0.0001"/>
         <mu2 value= "0.0001"/>

Commit message: md

File: description/lidar.xacro (robot description, xacro)
@@ -6,8 +6,13 @@
     <xacro:property name="lidar_offset_z"           value="0.12"/>
     <!-- Lidar -->
-    <joint name="lidar_joint" type="fixed">
+    <!-- <joint name="lidar_joint" type="fixed">
         <parent link="chasis"/>
         <child link="lidar_frame"/>
         <origin xyz="${lidar_offset_x} 0.0 ${lidar_offset_z}" rpy="0 0 0"/>
+    </joint> -->
+    <joint name="lidar_joint" type="fixed">
+        <parent link="base_link"/>
+        <child link="lidar_frame"/>
+        <origin xyz="0.133 0.0 0.105" rpy="0 0 0"/>
     </joint>
     <link name="lidar_frame">

Commit message: md 9/11

File: description/lidar.xacro (robot description, xacro)
@@ -9,10 +9,10 @@
         <parent link="chasis"/>
         <child link="lidar_frame"/>
-        <origin xyz="${lidar_offset_x} 0.0 ${lidar_offset_z}" rpy="0 0 0"/>
+        <origin xyz="${lidar_offset_x} 0.0 ${lidar_offset_z}" rpy="0 0 ${pi}"/>
     </joint> -->
     <joint name="lidar_joint" type="fixed">
         <parent link="base_link"/>
         <child link="lidar_frame"/>
-        <origin xyz="0.133 0.0 0.105" rpy="0 0 0"/>
+        <origin xyz="0.133 0.0 0.105" rpy="0 0 ${pi}"/>
     </joint>
     <link name="lidar_frame">

Commit message: md

File: description/lidar.xacro (robot description, xacro)
@@ -6,14 +6,14 @@
     <xacro:property name="lidar_offset_z"           value="0.12"/>
     <!-- Lidar -->
-    <!-- <joint name="lidar_joint" type="fixed">
+    <joint name="lidar_joint" type="fixed">
         <parent link="chasis"/>
         <child link="lidar_frame"/>
         <origin xyz="${lidar_offset_x} 0.0 ${lidar_offset_z}" rpy="0 0 ${pi}"/>
-    </joint> -->
-    <joint name="lidar_joint" type="fixed">
+    </joint>
+    <!-- <joint name="lidar_joint" type="fixed">
         <parent link="base_link"/>
         <child link="lidar_frame"/>
         <origin xyz="0.133 0.0 0.105" rpy="0 0 ${pi}"/>
-    </joint>
+    </joint> -->
     <link name="lidar_frame">
         <visual>
